File: hardware/Outputs.kicad_sch (KiCad schematic)
At the start: 0 parts

Commit message: Assign footprints to some components and improvements.
Parts:
- added D? (x4): LL4148, Diode_SMD:D_MiniMELF, symbol Diode:LL4148
- added J? (x8): Screw_Terminal_01x03, symbol Connector:Screw_Terminal_01x03
- added K? (x4): G2RL-2, Relay_THT:Relay_DPDT_Omron_G2RL-2, symbol Relay:G2RL-2
- added Q? (x4): 2N7002, Package_TO_SOT_SMD:SOT-23, symbol Transistor_FET:2N7002
- added R? (x4): 100K, symbol Device:R
Connections:
- new net: D?.2 (A), K?.A2, Q?.3 (D) (x4)
- new net: J?.3 (Pin_3), K?.11 (x4)
- new net: J?.1 (Pin_1), K?.12 (x4)
- new net: J?.2 (Pin_2), K?.14 (x4)
- new net: J?.3 (Pin_3), K?.21 (x4)
- new net: J?.1 (Pin_1), K?.22 (x4)
- new net: J?.2 (Pin_2), K?.24 (x4)
- new net +5V: D?.1 (K), D?.1 (K), D?.1 (K), D?.1 (K), K?.A1, K?.A1, K?.A1, K?.A1
- new net GND: Q?.2 (S), Q?.2 (S), Q?.2 (S), Q?.2 (S), R?.2, R?.2, R?.2, R?.2
- new net OUTPUT_ISO1: Q?.1 (G), R?.1
- new net OUTPUT_ISO2: Q?.1 (G), R?.1
- new net OUTPUT_ISO3: Q?.1 (G), R?.1
- new net OUTPUT_ISO4: Q?.1 (G), R?.1
Other:
- note added: "OUTPUTS ISOLATED"

Commit message: Improvements to schematic.
Other:
- company: (none) -> FEYTECH PTY LTD
- title: (none) -> MQTT Gateway
- moved on the sheet: D?, J?, K?, Q?, R?
